Commit message: 바퀴가 + 형태라서, 동그란 형태로 임의로 바꿨는데, nice하지 않음. linorobot에서 2wd or 4wd 를 가져와서 적용을 하면 좋겠음. ( fast_lio가 그나마 조금 그려짐 ) livox lidar 시뮬레이터가 gz sim용이 없어서, gpu lidar를 활용해 깨지지 않는 수준으로 그리는중

File: urdf/lidar_mid360_sensor.urdf.xacro (robot description, xacro)
@@ -58,13 +58,13 @@
             <horizontal>
               <samples>360</samples>
-              <resolution>1</resolution>
+              <resolution>0.1</resolution>
               <min_angle>-3.14159</min_angle>
               <max_angle>3.14159</max_angle>
             </horizontal>
             <vertical>
-              <samples>16</samples>
+              <samples>32</samples>
               <resolution>1</resolution>
-              <min_angle>-0.261</min_angle>
-              <max_angle>0.261</max_angle>
+              <min_angle>0.0</min_angle>
+              <max_angle>0.761</max_angle>
             </vertical>
           </scan>
@@ -77,5 +77,5 @@
             <type>gaussian</type>
             <mean>0.0</mean>
-            <stddev>0.01</stddev>
+            <stddev>0.001</stddev>
           </noise>
         </lidar>

File: urdf/robot.xacro.urdf (robot description, URDF)
Before this commit: robot diff_drive, 3 links, 2 joints
Joints:
- joint imu_joint: origin xyz=0 0 0.05 rpy=0.5 1.2 -1.17 -> xyz=0 0 0 rpy=0 0 0

File: urdf/wheel.xacro (robot description, xacro)
@@ -9,14 +9,20 @@
       </inertial>
       <visual>
-        <origin xyz="0.0 0.0 0.0" rpy="0 0 0"/>
+        <origin xyz="0.0 0.0 0.0" rpy="0.2 1.5707963 0"/>
+        <!-- <geometry>
+          <mesh filename="file://$(find nav2_outdoor_example)/urdf/meshes/wheel.stl" scale="0.001 0.001 0.001"/>
+        </geometry> -->
         <geometry>
-          <mesh filename="file://$(find nav2_outdoor_example)/urdf/meshes/wheel.stl" scale="0.001 0.001 0.001"/>
+          <cylinder radius="0.3" length="0.15"/>
         </geometry>
         <material name="silver"/>
       </visual>
       <collision>
-        <origin xyz="0.0 0.0 0.0" rpy="0 0 0"/>
+        <origin xyz="0.0 0.0 0.0" rpy="0.2 1.5707963 0"/>
+        <!-- <geometry>
+          <mesh filename="file://$(find nav2_outdoor_example)/urdf/meshes/wheel.stl" scale="0.001 0.001 0.001"/>
+        </geometry> -->
         <geometry>
-          <mesh filename="file://$(find nav2_outdoor_example)/urdf/meshes/wheel.stl" scale="0.001 0.001 0.001"/>
+          <cylinder radius="0.3" length="0.15"/>
         </geometry>
       </collision>
