Commit message: gps를 끄고, slam만으로 주행하는 테스트,

File: urdf/robot.xacro.urdf (robot description, URDF)
Before this commit: robot diff_drive, 2 links, 2 joints
Links:
- added link RGLLidar
Joints:
- added joint RGLLidar_to_base_joint: type fixed, parent base_link, child RGLLidar, origin xyz=0 0 0.5 rpy=0 0 0
